File: led-ring-v2/led-ring-v2/led-ring-v2.kicad_sch (KiCad schematic)
At the start: 40 parts, among them J1 Conn_01x02_Pin

Commit message: led-ring-v2.1
* fix polarity markings
* add lens circles to aid glue deposition
Parts:
- D1, D10, D11, D12, D13, D14, D15, D16, D17, D18, D19, D2, D20, D21, D3, D4, D5, D6, D7, D8, D9: footprint victor_strawlab:OSRAM_SFH_4715AS -> victor_strawlab:OSRAM_SFH_4715AS_with_LISA4
Changed lines of the file:
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@@
       (effects (font (size 1.27 1.27)) (justify left))
     )
-    (property "Footprint" "victor_strawlab:OSRAM_SFH_4715AS" (at 83.82 100.33 0)
+    (property "Footprint" "victor_strawlab:OSRAM_SFH_4715AS_with_LISA4" (at 83.82 100.33 0)
       (effects (font (size 1.27 1.27)) hide)
     )
@@
       (effects (font (size 1.27 1.27)) (justify left))
     )
-    (property "Footprint" "victor_strawlab:OSRAM_SFH_4715AS" (at 66.04 69.85 0)
+    (property "Footprint" "victor_strawlab:OSRAM_SFH_4715AS_with_LISA4" (at 66.04 69.85 0)
       (effects (font (size 1.27 1.27)) hide)
     )
@@
       (effects (font (size 1.27 1.27)) (justify left))
     )
-    (property "Footprint" "victor_strawlab:OSRAM_SFH_4715AS" (at 66.04 80.01 0)
+    (property "Footprint" "victor_strawlab:OSRAM_SFH_4715AS_with_LISA4" (at 66.04 80.01 0)
       (effects (font (size 1.27 1.27)) hide)
     )
@@
       (effects (font (size 1.27 1.27)) (justify left))
     )
-    (property "Footprint" "victor_strawlab:OSRAM_SFH_4715AS" (at 83.82 69.85 0)
+    (property "Footprint" "victor_strawlab:OSRAM_SFH_4715AS_with_LISA4" (at 83.82 69.85 0)
       (effects (font (size 1.27 1.27)) hide)
     )
@@
       (effects (font (size 1.27 1.27)) (justify left))
     )
-    (property "Footprint" "victor_strawlab:OSRAM_SFH_4715AS" (at 100.33 110.49 0)
+    (property "Footprint" "victor_strawlab:OSRAM_SFH_4715AS_with_LISA4" (at 100.33 110.49 0)
       (effects (font (size 1.27 1.27)) hide)
     )
@@
       (effects (font (size 1.27 1.27)) (justify left))
     )
-    (property "Footprint" "victor_strawlab:OSRAM_SFH_4715AS" (at 100.33 120.65 0)
+    (property "Footprint" "victor_strawlab:OSRAM_SFH_4715AS_with_LISA4" (at 100.33 120.65 0)
       (effects (font (size 1.27 1.27)) hide)
     )
@@
       (effects (font (size 1.27 1.27)) (justify left))
     )
-    (property "Footprint" "victor_strawlab:OSRAM_SFH_4715AS" (at 66.04 90.17 0)
+    (property "Footprint" "victor_strawlab:OSRAM_SFH_4715AS_with_LISA4" (at 66.04 90.17 0)
       (effects (font (size 1.27 1.27)) hide)
     )
@@
       (effects (font (size 1.27 1.27)) (justify left))
     )
-    (property "Footprint" "victor_strawlab:OSRAM_SFH_4715AS" (at 83.82 120.65 0)
+    (property "Footprint" "victor_strawlab:OSRAM_SFH_4715AS_with_LISA4" (at 83.82 120.65 0)
       (effects (font (size 1.27 1.27)) hide)
     )
@@
       (effects (font (size 1.27 1.27)) (justify left))
     )
-    (property "Footprint" "victor_strawlab:OSRAM_SFH_4715AS" (at 66.04 59.69 0)
+    (property "Footprint" "victor_strawlab:OSRAM_SFH_4715AS_with_LISA4" (at 66.04 59.69 0)
       (effects (font (size 1.27 1.27)) hide)
     )
@@
       (effects (font (size 1.27 1.27)) (justify left))
     )
-    (property "Footprint" "victor_strawlab:OSRAM_SFH_4715AS" (at 100.33 80.01 0)
+    (property "Footprint" "victor_strawlab:OSRAM_SFH_4715AS_with_LISA4" (at 100.33 80.01 0)
       (effects (font (size 1.27 1.27)) hide)
     )
@@
       (effects (font (size 1.27 1.27)) (justify left))
     )
-    (property "Footprint" "victor_strawlab:OSRAM_SFH_4715AS" (at 100.33 69.85 0)
+    (property "Footprint" "victor_strawlab:OSRAM_SFH_4715AS_with_LISA4" (at 100.33 69.85 0)
       (effects (font (size 1.27 1.27)) hide)
     )
@@
       (effects (font (size 1.27 1.27)) (justify left))
     )
-    (property "Footprint" "victor_strawlab:OSRAM_SFH_4715AS" (at 66.04 120.65 0)
+    (property "Footprint" "victor_strawlab:OSRAM_SFH_4715AS_with_LISA4" (at 66.04 120.65 0)
       (effects (font (size 1.27 1.27)) hide)
     )
@@
       (effects (font (size 1.27 1.27)) (justify left))
     )
-    (property "Footprint" "victor_strawlab:OSRAM_SFH_4715AS" (at 100.33 90.17 0)
+    (property "Footprint" "victor_strawlab:OSRAM_SFH_4715AS_with_LISA4" (at 100.33 90.17 0)
       (effects (font (size 1.27 1.27)) hide)
     )
@@
       (effects (font (size 1.27 1.27)) (justify left))
     )
-    (property "Footprint" "victor_strawlab:OSRAM_SFH_4715AS" (at 83.82 59.69 0)
+    (property "Footprint" "victor_strawlab:OSRAM_SFH_4715AS_with_LISA4" (at 83.82 59.69 0)
       (effects (font (size 1.27 1.27)) hide)
     )
@@
       (effects (font (size 1.27 1.27)) (justify left))
     )
-    (property "Footprint" "victor_strawlab:OSRAM_SFH_4715AS" (at 83.82 80.01 0)
+    (property "Footprint" "victor_strawlab:OSRAM_SFH_4715AS_with_LISA4" (at 83.82 80.01 0)
       (effects (font (size 1.27 1.27)) hide)
     )
@@
       (effects (font (size 1.27 1.27)) (justify left))
     )
-    (property "Footprint" "victor_strawlab:OSRAM_SFH_4715AS" (at 66.04 110.49 0)
+    (property "Footprint" "victor_strawlab:OSRAM_SFH_4715AS_with_LISA4" (at 66.04 110.49 0)
       (effects (font (size 1.27 1.27)) hide)
     )
@@
       (effects (font (size 1.27 1.27)) (justify left))
     )
-    (property "Footprint" "victor_strawlab:OSRAM_SFH_4715AS" (at 83.82 90.17 0)
+    (property "Footprint" "victor_strawlab:OSRAM_SFH_4715AS_with_LISA4" (at 83.82 90.17 0)
       (effects (font (size 1.27 1.27)) hide)
     )
@@
       (effects (font (size 1.27 1.27)) (justify left))
     )
-    (property "Footprint" "victor_strawlab:OSRAM_SFH_4715AS" (at 66.04 100.33 0)
+    (property "Footprint" "victor_strawlab:OSRAM_SFH_4715AS_with_LISA4" (at 66.04 100.33 0)
       (effects (font (size 1.27 1.27)) hide)
     )
@@
       (effects (font (size 1.27 1.27)) (justify left))
     )
-    (property "Footprint" "victor_strawlab:OSRAM_SFH_4715AS" (at 100.33 59.69 0)
+    (property "Footprint" "victor_strawlab:OSRAM_SFH_4715AS_with_LISA4" (at 100.33 59.69 0)
       (effects (font (size 1.27 1.27)) hide)
     )
@@
       (effects (font (size 1.27 1.27)) (justify left))
     )
-    (property "Footprint" "victor_strawlab:OSRAM_SFH_4715AS" (at 100.33 100.33 0)
+    (property "Footprint" "victor_strawlab:OSRAM_SFH_4715AS_with_LISA4" (at 100.33 100.33 0)
       (effects (font (size 1.27 1.27)) hide)
     )
@@
       (effects (font (size 1.27 1.27)) (justify left))
     )
-    (property "Footprint" "victor_strawlab:OSRAM_SFH_4715AS" (at 83.82 110.49 0)
-      (effects (font (size 1.27 1.27)) hide)
-    )
+    (property "Footprint" "victor_strawlab:OSRAM_SFH_4715AS_with_LISA4" (at 83.82 110.49 0)
+      (effects (font (size 1.27 1.27)) hide)
+    )
